Commit message: feat: add kuka_trajectory_logger node to capture MoveIt2 planned trajectories to CSV

File: ros2_ws/src/kuka_kr6_support/urdf/environment.xacro (robot description, xacro)
@@ -118,5 +118,11 @@
   <link name="gripper_env_link">
     <visual>
-      <origin xyz="0 0 0" rpy="0 0 0"/>
+      <!-- Ajuste SOLO de la malla (el frame del link NO se mueve):
+           eje longitudinal del STL (+X mesh) alineado con +Z del link,
+           eje del collar trasero (Y=39.04mm, Z=19.2mm del STL) sobre el eje del flange,
+           cara ESTRUCTURAL de la placa base (x=8.858mm del STL) al ras del flange.
+           El collar y los pasadores (x<8.858mm) quedan alojados dentro del
+           cilindro del flange (r=18.2mm < 20mm, 8.8mm < 13.5mm de largo). -->
+      <origin xyz="0.0192 -0.03904 -0.008858" rpy="0 -1.5708 0"/>
       <geometry>
         <mesh filename="package://kuka_kr6_support/meshes/environment/gripper.stl" scale="1 1 1"/>
@@ -125,5 +131,7 @@
     </visual>
     <collision>
-      <origin xyz="0 0 0" rpy="0 0 0"/>
+      <!-- Volumen fisico del gripper para MoveIt2: misma malla y EXACTAMENTE la
+           misma transformacion que <visual>, para que collision y visual coincidan. -->
+      <origin xyz="0.0192 -0.03904 -0.008858" rpy="0 -1.5708 0"/>
       <geometry>
         <mesh filename="package://kuka_kr6_support/meshes/environment/gripper.stl" scale="1 1 1"/>
@@ -142,5 +150,8 @@
   <link name="cubo_env_link">
     <visual>
-      <origin xyz="0 0 0" rpy="0 0 0"/>
+      <!-- Ajuste SOLO visual: centra el cubo (30mm) entre las mordazas, sobre el eje
+           del gripper y a 118mm del flange (zona de agarre; puntas a 144mm).
+           Compensa el offset del cubo_env_joint, que NO se toca. -->
+      <origin xyz="0.005 0 0.083" rpy="0 0 0"/>
       <geometry>
         <mesh filename="package://kuka_kr6_support/meshes/environment/cubo.stl" scale="1 1 1"/>

Commit message: refactor: realign environment base and table meshes by updating URDF origins and synchronizing mesh files

File: ros2_ws/src/kuka_kr6_support/urdf/environment.xacro (robot description, xacro)
@@ -70,5 +70,10 @@
   <link name="base_env_link">
     <visual>
-      <origin xyz="0 0 0" rpy="0 0 0"/>
+      <!-- Ajuste SOLO de la malla (el frame del link, el joint y el KUKA NO se mueven):
+           traslacion vertical PURA de dz = -0.030334282 m en Z de base_link,
+           expresada en el frame del link como R^T*(0,0,dz) con rpy = 1.57 0 0.
+           Resultado: Z_max(base.stl) = 0.000 m = cara inferior de la base del KUKA
+           (contacto exacto, sin penetracion). X, Y y rpy quedan intactos. -->
+      <origin xyz="0 -0.030334272 -0.000024156" rpy="0 0 0"/>
       <geometry>
         <mesh filename="package://kuka_kr6_support/meshes/environment/base.stl" scale="1 1 1"/>
@@ -77,5 +82,6 @@
     </visual>
     <collision>
-      <origin xyz="0 0 0" rpy="0 0 0"/>
+      <!-- Mismo desplazamiento que <visual>: collision y visual siguen superpuestos. -->
+      <origin xyz="0 -0.030334272 -0.000024156" rpy="0 0 0"/>
       <geometry>
         <mesh filename="package://kuka_kr6_support/meshes/environment/base.stl" scale="1 1 1"/>
@@ -94,5 +100,10 @@
   <link name="mesa_env_link">
     <visual>
-      <origin xyz="0 0 0" rpy="0 0 0"/>
+      <!-- Ajuste SOLO de la malla (el frame del link, el joint y el KUKA NO se mueven):
+           traslacion vertical PURA de dz = -0.030413915 m en Z de base_link,
+           expresada en el frame del link como R^T*(0,0,dz) con rpy = 1.57 0 1.57.
+           Resultado: Z_min(patas mesa) = Z_min(base.stl) = -0.560334282 m,
+           es decir ambas apoyan en el mismo plano. X, Y y rpy quedan intactos. -->
+      <origin xyz="0 -0.030413905 -0.000024219" rpy="0 0 0"/>
       <geometry>
         <mesh filename="package://kuka_kr6_support/meshes/environment/mesa.stl" scale="1 1 1"/>
@@ -101,5 +112,6 @@
     </visual>
     <collision>
-      <origin xyz="0 0 0" rpy="0 0 0"/>
+      <!-- Mismo desplazamiento que <visual>: collision y visual siguen superpuestos. -->
+      <origin xyz="0 -0.030413905 -0.000024219" rpy="0 0 0"/>
       <geometry>
         <mesh filename="package://kuka_kr6_support/meshes/environment/mesa.stl" scale="1 1 1"/>

Commit message: feat: add configurable tool selection between gripper and marker via launch argument

File: ros2_ws/src/kuka_kr6_support/urdf/environment.xacro (robot description, xacro)
@@ -41,4 +41,10 @@
   <xacro:property name="cubo_P"       default="0"/>
   <xacro:property name="cubo_Y"       default="0"/>
+  <!-- ── Tool selection: gripper (default) | marker ──────────────── -->
+  <!-- Selecciona SOLO la geometria representada dentro de gripper_env_link.
+       No crea links, joints ni frames nuevos: la cadena cinematica, el flange
+       y el TCP son identicos para ambos valores.                              -->
+  <xacro:arg name="tool" default="gripper"/>
+  <xacro:property name="tool" value="$(arg tool)"/>
   <!-- ── Robot vertical offset (raises KUKA relative to env) ───── -->
   <!-- Increase to raise the robot above the pedestal/mesa          -->
@@ -129,4 +135,8 @@
   <!-- ============================================================ -->
   <link name="gripper_env_link">
+    <!-- Herramienta seleccionable:  tool:=gripper (por defecto) | tool:=marker
+         Las dos ramas son mutuamente excluyentes; comparten este mismo link,
+         el mismo frame y el mismo gripper_env_joint (que NO se toca). -->
+    <xacro:if value="${tool == 'gripper'}">
     <visual>
       <!-- Ajuste SOLO de la malla (el frame del link NO se mueve):
@@ -150,4 +160,29 @@
       </geometry>
     </collision>
+    </xacro:if>
+    <xacro:if value="${tool == 'marker'}">
+    <visual>
+      <!-- Ajuste SOLO de la malla (mismo frame que el gripper, sin tocar el joint):
+           eje longitudinal del STL (+Y mesh, 0..147mm) alineado con +Z del link,
+           eje de la placa de montaje (X=22.5mm, Z=22.5mm del STL) sobre el eje
+           del flange, y cara de montaje (disco de 45mm en y=0) al ras del flange.
+           El yaw de 2.35619 rad (135 deg) es un giro PURO sobre el eje de la
+           herramienta: deja el talon de montaje arriba y no altera ni el apoyo
+           ni la coaxialidad. -->
+      <origin xyz="0 -0.0318198 0" rpy="1.5708 0 2.35619"/>
+      <geometry>
+        <mesh filename="package://kuka_kr6_support/meshes/environment/marker.stl" scale="1 1 1"/>
+      </geometry>
+      <material name="env_gray"/>
+    </visual>
+    <collision>
+      <!-- Volumen fisico del marcador para MoveIt2: misma malla y EXACTAMENTE la
+           misma transformacion que su <visual>. -->
+      <origin xyz="0 -0.0318198 0" rpy="1.5708 0 2.35619"/>
+      <geometry>
+        <mesh filename="package://kuka_kr6_support/meshes/environment/marker.stl" scale="1 1 1"/>
+      </geometry>
+    </collision>
+    </xacro:if>
   </link>
   <joint name="gripper_env_joint" type="fixed">
@@ -161,4 +196,9 @@
   <!-- ============================================================ -->
   <link name="cubo_env_link">
+    <!-- El cubo es la pieza que sujeta el gripper: solo se representa con
+         tool:=gripper. Con tool:=marker el link y su cubo_env_joint siguen
+         existiendo (frame y TF intactos, referencias del SRDF validas) pero
+         no llevan geometria, asi que no se ve nada. -->
+    <xacro:if value="${tool == 'gripper'}">
     <visual>
       <!-- Ajuste SOLO visual: centra el cubo (30mm) entre las mordazas, sobre el eje
@@ -177,4 +217,5 @@
       </geometry>
     </collision>
+    </xacro:if>
   </link>
   <joint name="cubo_env_joint" type="fixed">
